File: Kicad-Stamp-Board/Stamp-STM32F.kicad_pcb (KiCad board)
At the start: 2 copper layers, 65.4 x 43.7 mm, 33 parts, among them J1 Conn_01x25, J2 Conn_01x25, J3 Conn_01x04, J4 BOOT1, SW1 Reset, SW2 BOOT, U1 STM32F103RET6, U2 ICL3221, Y1 32.768KHz

Commit message: Small mods to PCB and README. Gerbers.
Parts:
- moved J1 1.27 mm to (177.8, 76.2)
Routing:
- net PA8: track 30.0 -> 28.1 mm
- net RESET: track 88.5 -> 87.2 mm
- net PA0: track 51.2 -> 49.9 mm
- net PA3: track 57.0 -> 55.7 mm
- net PA4: track 58.0 -> 56.8 mm
- net PA2: track 55.1 -> 53.8 mm
- net PA1: track 52.2 -> 51.0 mm
- net PB6: track 40.2 -> 39.0 mm
- net PB5: track 39.2 -> 38.0 mm
- net PB4: track 38.3 -> 37.1 mm
- net PB3: track 35.6 -> 34.4 mm
- net PB2: track 80.6 -> 79.4 mm
- net 3.3V: track 173.3 -> 172.1 mm
- net PA5: track 59.1 -> 57.9 mm
- net PA6: track 60.1 -> 59.5 mm
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Other:
- board size 65.4 x 43.7 mm -> 65 x 41.5 mm
- board text added: "STM32F STAMP Board K Sarkies 09/12/2017 Version 0.0"
